File: MTC_DRIVER_PAYLOAD_BRD/EXAMPLE_BRD/_autosave-XTB.kicad_pcb (KiCad board)
At the start: 2 copper layers, 15.2 x 25.4 mm, 23 parts, among them J1 Conn_01x09, J2 Conn_01x09, J3 Conn_01x01, J4 Conn_01x01, U1 LM4120-1P8DBV, U2 M-QFN28_B, U4 Value, U5 Value

Commit message: pulled sample board
Connections:
- net /3.3V renamed +3V3
- net /GND renamed GND
- J1 pad 2: Net-(J1-Pad2) -> unconnected-(J1-Pin_2-Pad2)
- J2 pad 1: Net-(J2-Pad1) -> unconnected-(J2-Pin_1-Pad1)
- J2 pad 2: Net-(J2-Pad2) -> unconnected-(J2-Pin_2-Pad2)
- J2 pad 3: Net-(J2-Pad3) -> unconnected-(J2-Pin_3-Pad3)
- J2 pad 4: Net-(J2-Pad4) -> unconnected-(J2-Pin_4-Pad4)
- J2 pad 7: Net-(J2-Pad7) -> unconnected-(J2-Pin_7-Pad7)
- U1 pad 1: Net-(U1-Pad1) -> unconnected-(U1-REF-Pad1)
- U2 pad 10: Net-(U2-Pad10) -> unconnected-(U2-Pad10)
- U2 pad 11: Net-(U2-Pad11) -> unconnected-(U2-Pad11)
- U2 pad 12: Net-(U2-Pad12) -> unconnected-(U2-Pad12)
- U2 pad 14: Net-(U2-Pad14) -> unconnected-(U2-Pad14)
- U2 pad 7: Net-(U2-Pad7) -> unconnected-(U2-Pad7)
- U2 pad 9: Net-(U2-Pad9) -> unconnected-(U2-Pad9)
