File: TORQUERS/V1_BOARDS/XY_PANEL/Xpanel_V1_final.kicad_pcb (KiCad board)
At the start: 4 copper layers, 82.6 x 98 mm, 99 parts, among them J1 F3311A7H121014E200, J2 F3311A7H121014E200, Q1 BSS138, Q10 MBT2222ADW1T1, Q11 BSS138, Q12 MBT2222ADW1T1, Q2 BSS138, Q3 BSS138, Q4 MBT2222ADW1T1, Q5 BSS138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

Commit message: made changes with feedback
Parts:
- removed L1, L2: TBD, Inductor_SMD:L_0603_1608Metric
- J1, J2: footprint F3311A7H121008E200:F3311A7H121014E200 -> AA_AUTO_LOADER:F3311A7H121014E200
- moved D2 5.87 mm to (156.1, 68.6)
- moved D1 5.69 mm to (161.1, 72.0)
Connections:
- JP2 pad 3: /SUN_SENSOR/+3.3v -> +3.3V
- U2 pad 1: Net-(U2-OUT2) -> Net-(JP3-A)
- U2 pad 3: Net-(U2-OUT1) -> Net-(JP3-B)
- U3 pad 1: /SUN_SENSOR/+3.3v -> +3.3V
Routing:
- net +3.3V: track 189.5 -> 207.0 mm, vias 8 -> 9
- net Net-(JP3-B): track 4.69 -> 20.6 mm
- net Net-(U2-OUT1): track 14.0 -> 0.00 mm
- net Net-(JP3-A): track 10.1 -> 22.3 mm
- net Net-(U2-OUT2): track 10.6 -> 0.00 mm
- net GND: track 375.8 -> 383.4 mm
- net /solar_panel_electronics/3224_vout: track 38.1 -> 32.2 mm
- net /solar_panel_electronics/7023_vout: track 18.4 -> 22.3 mm
- net Net-(D1-K): track 57.8 -> 54.4 mm
- net /SUN_SENSOR/+3.3v: track 2.14 -> 0.00 mm
- net SCL_SUN: track 38.1 -> 39.6 mm
