File: PyCubed/Burn_Wires.kicad_sch (KiCad schematic)
At the start: 4 parts, among them J19 F3311A7H121014E200, J4 1985807

Commit message: PyCubed Schematic Finalized
Parts:
- added J19 (x4): F3311A7H121014E200, F3311A7H121014E200, symbol SamacSys_Parts:F3311A7H121014E200
Connections:
- net 3.3V: now also J19.10, J19.10, J19.10, J19.10, J19.5, J19.5, J19.5, J19.5
- net GND: now also J19.11, J19.11, J19.11, J19.11, J19.4, J19.4, J19.4, J19.4, J19.MP1, J19.MP1, J19.MP1, J19.MP1, J19.MP2, J19.MP2, J19.MP2, J19.MP2
- net SCL2: now also J19.6, J19.6, J19.6, J19.6, J19.9, J19.9, J19.9, J19.9
- net SDA2: now also J19.7, J19.7, J19.7, J19.7, J19.8, J19.8, J19.8, J19.8
- net VBATT: now also J19.12, J19.12, J19.12, J19.12, J19.13, J19.13, J19.13, J19.13, J19.2, J19.2, J19.2, J19.2, J19.3, J19.3, J19.3, J19.3
- net VSOLAR: now also J19.1, J19.1, J19.1, J19.1, J19.14, J19.14, J19.14, J19.14
Other:
- note added: "X+"
- note added: "X-"
- note added: "Y+"
- note added: "Y-"

Commit message: Mainboard Final Design
Updated BMS
Parts:
- added J4: 1985807, mainboard:SCREWTERMINAL-3.5MM-2_LOCK, symbol mainboard:M023.5MM_LOCK
Connections:
- net GND: now also J4.1, J4.2
- net VBATT: no longer J19.12, J19.12, J19.13, J19.13, J19.2, J19.2, J19.3, J19.3
Changed lines of the file:
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@@
   (junction (at 45.72 161.29) (diameter 0) (color 0 0 0 0)
   )
+  (junction (at 201.93 58.42) (diameter 0) (color 0 0 0 0)
+  )
   (junction (at 137.16 68.58) (diameter 0) (color 0 0 0 0)
   )
@@
     (stroke (width 0) (type default))
   )
+  (wire (pts (xy 201.93 58.42) (xy 201.93 59.69))
+    (stroke (width 0) (type default))
+  )
   (wire (pts (xy 133.35 162.56) (xy 130.81 162.56))
     (stroke (width 0) (type default))
@@
   )
   (wire (pts (xy 130.81 167.64) (xy 143.51 167.64))
+    (stroke (width 0) (type default))
+  )
+  (wire (pts (xy 201.93 55.88) (xy 201.93 58.42))
     (stroke (width 0) (type default))
   )
@@
     )
   )
-  (global_label "VBATT" (shape bidirectional) (at 123.19 114.3 0)
-    (effects (font (size 1.27 1.27)) (justify left))
-    (property "Intersheetrefs" "${INTERSHEET_REFS}" (at 123.19 114.3 0)
-      (effects (font (size 1.27 1.27)) hide)
-    )
-  )
   (global_label "SDA2" (shape bidirectional) (at 123.19 124.46 0)
     (effects (font (size 1.27 1.27)) (justify left))
@@
     )
   )
-  (global_label "VBATT" (shape bidirectional) (at 74.93 110.49 0)
-    (effects (font (size 1.27 1.27)) (justify left))
-    (property "Intersheetrefs" "${INTERSHEET_REFS}" (at 74.93 110.49 0)
-      (effects (font (size 1.27 1.27)) hide)
-    )
-  )
   (global_label "VBATT" (shape bidirectional) (at 73.66 186.69 0)
     (effects (font (size 1.27 1.27)) (justify left))
@@
     )
   )
-  (global_label "VBATT" (shape bidirectional) (at 123.19 139.7 0)
-    (effects (font (size 1.27 1.27)) (justify left))
-    (property "Intersheetrefs" "${INTERSHEET_REFS}" (at 123.19 139.7 0)
-      (effects (font (size 1.27 1.27)) hide)
-    )
-  )
   (global_label "SCL2" (shape bidirectional) (at 236.22 123.19 0)
     (effects (font (size 1.27 1.27)) (justify left))
@@
     )
   )
-  (global_label "VBATT" (shape bidirectional) (at 123.19 111.76 0)
-    (effects (font (size 1.27 1.27)) (justify left))
-    (property "Intersheetrefs" "${INTERSHEET_REFS}" (at 123.19 111.76 0)
-      (effects (font (size 1.27 1.27)) hide)
-    )
-  )
   (global_label "VBATT" (shape bidirectional) (at 133.35 190.5 0)
     (effects (font (size 1.27 1.27)) (justify left))
@@
     )
   )
-  (global_label "VBATT" (shape bidirectional) (at 123.19 137.16 0)
-    (effects (font (size 1.27 1.27)) (justify left))
-    (property "Intersheetrefs" "${INTERSHEET_REFS}" (at 123.19 137.16 0)
-      (effects (font (size 1.27 1.27)) hide)
-    )
-  )
   (global_label "ENAB_BURN1" (shape bidirectional) (at 113.03 48.26 0)
     (effects (font (size 1.27 1.27)) (justify left))
@@
     )
   )
-  (global_label "VBATT" (shape bidirectional) (at 74.93 138.43 0)
-    (effects (font (size 1.27 1.27)) (justify left))
-    (property "Intersheetrefs" "${INTERSHEET_REFS}" (at 74.93 138.43 0)
-      (effects (font (size 1.27 1.27)) hide)
-    )
-  )
   (global_label "SCL2" (shape bidirectional) (at 179.07 121.92 0)
     (effects (font (size 1.27 1.27)) (justify left))
@@
     )
   )
-  (global_label "VBATT" (shape bidirectional) (at 74.93 135.89 0)
-    (effects (font (size 1.27 1.27)) (justify left))
-    (property "Intersheetrefs" "${INTERSHEET_REFS}" (at 74.93 135.89 0)
-      (effects (font (size 1.27 1.27)) hide)
-    )
-  )
   (global_label "VSOLAR" (shape bidirectional) (at 133.35 160.02 0)
     (effects (font (size 1.27 1.27)) (justify left))
@@
     (effects (font (size 1.27 1.27)) (justify left))
     (property "Intersheetrefs" "${INTERSHEET_REFS}" (at 179.07 137.16 0)
-      (effects (font (size 1.27 1.27)) hide)
-    )
-  )
-  (global_label "VBATT" (shape bidirectional) (at 74.93 113.03 0)
-    (effects (font (size 1.27 1.27)) (justify left))
-    (property "Intersheetrefs" "${INTERSHEET_REFS}" (at 74.93 113.03 0)
       (effects (font (size 1.27 1.27)) hide)
     )
@@
     )
   )
+  (symbol (lib_id "mainboard:M023.5MM_LOCK") (at 194.31 55.88 0) (mirror x) (unit 1)
+    (in_bom yes) (on_board yes) (dnp no)
+    (property "Reference" "J4" (at 186.69 54.61 0)
+      (effects (font (size 1.4986 1.4986)) (justify left bottom))
+    )
+    (property "Value" "1985807" (at 189.23 50.8 0)
+      (effects (font (size 1.4986 1.4986)) (justify left bottom))
+    )
+    (property "Footprint" "mainboard:SCREWTERMINAL-3.5MM-2_LOCK" (at 194.31 55.88 0)
+      (effects (font (size 1.27 1.27)) hide)
+    )
+    (property "Datasheet" "https://www.mouser.com/datasheet/2/324/4/1985807-1458929.pdf" (at 194.31 55.88 0)
+      (effects (font (size 1.27 1.27)) hide)
+    )
+    (property "Description" "2-pin Screw Terminal - Side Entry" (at 194.31 55.88 0)
+      (effects (font (size 1.27 1.27)) hide)
+    )
+    (property "Flight" "1985807" (at 194.31 55.88 0)
+      (effects (font (size 1.27 1.27)) hide)
+    )
+    (property "Manufacturer_Name" "Phoenix Contact" (at 194.31 55.88 0)
+      (effects (font (size 1.27 1.27)) hide)
+    )
+    (property "Manufacturer_Part_Number" "1985807" (at 186.69 57.15 0)
+      (effects (font (size 1.27 1.27)) hide)
+    )
+    (property "Proto" "1985807" (at 194.31 55.88 0)
+      (effects (font (size 1.27 1.27)) hide)
+    )
+    (pin "1")
+    (pin "2")
+    (instances
+      (project "mainboard"
+        (path "/351761a0-c9d1-4ae2-83c5-bde0949aa75f/00000000-0000-0000-0000-00005cec60eb"
+          (reference "J4") (unit 1)
+        )
+        (path "/351761a0-c9d1-4ae2-83c5-bde0949aa75f"
+          (reference "JP?") (unit 1)
+        )
+        (path "/351761a0-c9d1-4ae2-83c5-bde0949aa75f/00000000-0000-0000-0000-00005cec6476"
+          (reference "J8") (unit 1)
+        )
+      )
+    )
+  )
   (symbol (lib_id "SamacSys_Parts:F3311A7H121014E200") (at 208.28 110.49 0) (unit 1)
     (in_bom yes) (on_board yes) (dnp no) (fields_autoplaced)
@@
         )
         (path "/351761a0-c9d1-4ae2-83c5-bde0949aa75f"
+          (reference "#GND?") (unit 1)
+        )
+      )
+    )
+  )
+  (symbol (lib_id "mainboard:GND") (at 201.93 62.23 0) (unit 1)
+    (in_bom yes) (on_board yes) (dnp no)
+    (property "Reference" "#GND030" (at 201.93 62.23 0)
+      (effects (font (size 1.27 1.27)) hide)
+    )
+    (property "Value" "GND" (at 199.39 64.77 0)
+      (effects (font (size 1.4986 1.4986)) (justify left bottom))
+    )
+    (property "Footprint" "" (at 201.93 62.23 0)
+      (effects (font (size 1.27 1.27)) hide)
+    )
+    (property "Datasheet" "" (at 201.93 62.23 0)
+      (effects (font (size 1.27 1.27)) hide)
+    )
+    (pin "1")
+    (instances
+      (project "mainboard"
+        (path "/351761a0-c9d1-4ae2-83c5-bde0949aa75f/00000000-0000-0000-0000-00005cec6476"
+          (reference "#GND030") (unit 1)
+        )
+        (path "/351761a0-c9d1-4ae2-83c5-bde0949aa75f"
