File: PyCubed/Bus_Protection.kicad_sch (KiCad schematic)
At the start: 83 parts, among them Q11 MMDT2907, Q12 BSS138DWQ-7, Q13 BSS138DWQ-7, Q15 MBT2222ADW1T1, Q16 MBT2222ADW1T1, Q17 BSS138DWQ-7, Q18 BSS138DWQ-7, Q19 BSS138DWQ-7, Q20 MBT2222ADW1T1, Q28 MBT2222ADW1T1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

Commit message: Mainboard Final Design
Updated BMS
Changed lines of the file:
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@@
     (effects (font (size 2.159 2.159)) (justify left bottom))
   )
-  (text "Bus Protection - Bypass Jumpers" (at 59.69 172.72 0)
+  (text "Bus Protection - Bypass Jumpers" (at 46.99 171.45 0)
     (effects (font (size 2.159 2.159)) (justify left bottom))
   )
