File: PyCubed/Connectors.kicad_sch (KiCad schematic)
At the start: 17 parts, among them J1 503182-1852, J13 USB_C_Receptacle_USB2.0, J16 1985807, J17 1985807, J18 1985807, J2 Conn_01x05, J3 1985807, J4 1985807, U8 MR25H40MDF

Commit message: Mainboard Final Design
Updated BMS
Parts:
- added C26: 4.7nF, Capacitor_SMD:C_0603_1608Metric, symbol Device:C_Small
- added H1, H2, H3, H4: MountingHole_Pad, MountingHole:MountingHole_3.2mm_M3_DIN965_Pad, symbol Mechanical:MountingHole_Pad
- added R23: 1M, Resistor_SMD:R_0603_1608Metric, symbol Device:R_US
- added R28, R29: 22R, Resistor_SMD:R_0603_1608Metric, symbol Device:R_US
- added U10: USBLC6-2SC6, Package_TO_SOT_SMD:SOT-23-6, symbol Power_Protection:USBLC6-2SC6
Connections:
- net GND: now also H1.1, H2.1, H3.1, H4.1
- net GNDREF: now also C26.1, R23.1, U10.2 (GND); no longer J13.S1 (SHIELD)
- net USB_D+: now also U10.1 (I/O1); no longer J13.A6 (D+), J13.B6 (D+)
- net USB_D-: now also U10.3 (I/O2); no longer J13.A7 (D-), J13.B7 (D-)
- net VBUS_IN: now also U10.5 (VBUS)
- net VCHRG: no longer J16.1
- new net: C26.2, J13.S1 (SHIELD), R23.2
- new net DBus+: J13.A7 (D-), J13.B7 (D-), R28.2
- new net DBus-: J13.A6 (D+), J13.B6 (D+), R29.1
- new net DN: R29.2, U10.4 (I/O2)
- new net DP: R28.1, U10.6 (I/O1)
- new net VSYS: J16.1
Other:
- note added: "Mounting Holes"
- note added: "USB ESD Protection"
