File: PyCubed/Power.kicad_sch (KiCad schematic)
At the start: 69 parts, among them J14 Conn_01x06, Q1 IRLML2803, Q2 MBT2222ADW1T1, Q22 NDS8434, Q3 MBT2222ADW1T1, U17 BQ25883RGER, U21 TPS7A4501DCQT, U4 ADM1176-1ARMZ-R7, U5 TPS54226PWPRPWP14_2P31X2P46-L, U6 LTC4121, U7 KF50BD-TR

Commit message: Mainboard Final Design
Updated BMS
Parts:
- removed C22: 10uF, Capacitor_SMD:C_0603_1608Metric, symbol mainboard:10UF-0603-6.3V-20%
- removed C23: 2.2uF, Capacitor_SMD:C_0603_1608Metric, symbol mainboard:2.2UF-0603-10V-20%
- removed C25: 22nF, Capacitor_SMD:C_0603_1608Metric, symbol mainboard:2.2NF_2200PF-0603-50V-10%
- removed C28: 22uF, Capacitor_SMD:C_0603_1608Metric, symbol mainboard:0.1UF-0603-25V-5%
- removed C45: 0.1uF, Capacitor_SMD:C_0603_1608Metric, symbol Device:C_Small
- removed D2: DFLS130L, mainboard:PWRDI-123, symbol mainboard:DFLS130L
- removed JP6: Jumper_3_Bridged12, mainboard:SolderJumper-3_P1.3mm_Bridged12_RoundedPad1.0x1.5mm, symbol mainboard-rescue:Jumper_3_Bridged12-Jumper
- removed L3: 33uH, Inductor_SMD:L_1812_4532Metric, symbol Device:L
- removed Q1: IRLML2803, mainboard:SOT-23, symbol mainboard:IRLML2803TRPBF
- removed Q22: NDS8434, mainboard:NDS8434, symbol mainboard:NDS8434
- removed R10: 0, Resistor_SMD:R_0603_1608Metric, symbol mainboard:R-US_R0603
- removed R11: 787K, Resistor_SMD:R_0603_1608Metric, symbol mainboard:R-US_R0603
- removed R12: 121K, Resistor_SMD:R_0603_1608Metric, symbol mainboard:R-US_R0603
- removed R16: 845K, Resistor_SMD:R_0603_1608Metric, symbol mainboard:R-US_R0603
- removed R17, R18: 100k, Resistor_SMD:R_0603_1608Metric, symbol mainboard:R-US_R0603
- removed R19: 2.1M, Resistor_SMD:R_0603_1608Metric, symbol mainboard:R-US_R0603
- removed R20: 3.01K, Resistor_SMD:R_0603_1608Metric, symbol mainboard:R-US_R0603
- removed R21: 10K, Resistor_SMD:R_0603_1608Metric, symbol mainboard:R-US_R0603
- removed R22: 4.7K, Resistor_SMD:R_0603_1608Metric, symbol mainboard:R-US_R0603
- removed R23: 3.3K, Resistor_SMD:R_0603_1608Metric, symbol mainboard:R-US_R0603
- removed R9: 107K, Resistor_SMD:R_0603_1608Metric, symbol mainboard:R-US_R0603
- removed U6: LTC4121, mainboard:QFN-16-PAD, symbol mainboard:LTC4121
- removed U7: KF50BD-TR, mainboard:SOIC127P600X175-8N, symbol mainboard:KF50BD-TR
- added C22, C23: 47uF 25V, CAPC3225X279N, symbol SamacSys_Parts:12103D476MAT2A
- added C25: 1uF 25V, CAPC3225X170N, symbol SamacSys_Parts:VJ1210Y105KXXAT
- added C28: 10uF 25V, CAPC3225X230N, symbol SamacSys_Parts:C3225X7R1E106K250AC
- added C65: 10uF, Capacitor_SMD:C_0603_1608Metric, symbol mainboard:10UF-0603-6.3V-20%
- added C68: 10u 35V, CAPC3216X180N, symbol SamacSys_Parts:MLASU31LBB5106KTNA01
- added C69: 0.1u 10V, CAPC1608X87N, symbol SamacSys_Parts:C0603T104K8RAC7867
- added C70, C74: 0.015uF 50V, C0805, symbol SamacSys_Parts:C0805C153F5GALTU
- added C72, C73: 4.7uF 6.3V, CAPC1005X80N, symbol SamacSys_Parts:KAM05CT70J475KH
- added C77, C78: 0.22uF 16V, CAPC1005X70N, symbol SamacSys_Parts:GRT155R61A106ME13J
- added D7: V2NM153-M3_I, SE20NJM3H, symbol SamacSys_Parts:V2NM153-M3_I
- added D8: VSSAF5L45-M3_6A, SODFL5226X100N, symbol SamacSys_Parts:VSSAF5L45-M3_6A
- added IC3: MAX77961BEFV12+, MAX77961EFV06T, symbol SamacSys_Parts:MAX77961BEFV12+
- added L6: 1.5uH, INDPM5350X300N, symbol SamacSys_Parts:MPX1D0530L1R5
- added R153: 10m 3W, RESC3264X70N, symbol SamacSys_Parts:LTR100LJZPFU10L0
- added R154, R155: 10 1/4W, RESC2013X65N, symbol SamacSys_Parts:RL1220S-100-F
- added R157, R158: 200k 1/4W, RCC0805_e3, symbol SamacSys_Parts:RCC0805200KFKEA
- added R159: ERJ-2RKF6982X, ERJ2RKD1004X, symbol SamacSys_Parts:ERJ-2RKF6982X
- added R160, R161, R162, R163: 10K, Resistor_SMD:R_0603_1608Metric, symbol Device:R_US
- added R164, R165: 69.8k 1/4W, ERA8KEB1004V, symbol SamacSys_Parts:ERA-8VRW6982V
- added R166: 178k 1/4W, RESC3216X50N, symbol SamacSys_Parts:RG3216N-1783-D-T5
- added R167: 86.6k 1/4W, RESC3216X70N, symbol SamacSys_Parts:ERA-8ARB8662V
- added R9: ERJ-UP3J4R7V, ERJUP3, symbol SamacSys_Parts:ERJ-UP3J4R7V
Connections:
- net V_RF is gone; now on net VCC_RF1: C43.2, R55.1, U21.4 (OUT)
- net GND: now also C22.1, C23.1, C25.1, C28.1, C65.1, C68.1, C70.1, C72.2, C73.2, C74.1, IC3.10 (BATSN), IC3.14 (SCL), IC3.15 (SDA), IC3.18 (INTB), IC3.20 (GND), IC3.4 (PGND), R159.1, R161.2, R162.2, R164.1, R165.1, R166.1, R167.1
- net THM: now also IC3.13 (THM), R160.1; no longer R34.2, R35.2, R46.2, U17.7 (TS)
- net VBATT: now also C65.2
- net VCHRG: now also C28.2, D8.2 (A), IC3.11 (BATSP), IC3.12 (BATT_1), IC3.31 (BATT_2)
- net VSOLAR: now also D7.2 (A)
- new net: C68.2, IC3.2 (CHGIN), R153.2, R154.2 (R2)
- new net: D7.1 (K_1), D7.3 (K_2), R153.1, R155.2 (R2)
- new net: IC3.22 (CNFG), R159.2
- new net AVL: C72.1, IC3.26 (AVL), R160.2, R9.1
- new net BST1: C78.1, IC3.1 (BST1)
- new net BST2: C77.1, IC3.9 (BST2)
- new net CSINN: C69.2, C70.2, IC3.30 (CSINN), R154.1 (R1)
- new net CSINP: C69.1, C74.2, IC3.29 (CSINP), R155.1 (R1)
- new net DISQBAT: IC3.8 (DISQBAT), R162.1
- new net INLIM: IC3.21 (INLIM), R164.2
- new net INOKB: IC3.17 (INOKB), R157.1
- new net ISET: IC3.23 (ISET), R165.2
- new net ITO: IC3.25 (ITO), R166.2
- new net LX1: C78.2, IC3.3 (LX1), L6.2
- new net LX2: C77.2, IC3.5 (LX2), L6.1
- new net OTGEN: IC3.7 (OTGEN), R161.1
- new net PVL: C73.1, IC3.27 (PVL), R157.2, R158.2, R163.2, R9.2
- new net STAT1: IC3.16 (STAT), R158.1
- new net STBY: IC3.28 (STBY), R163.1
- new net TS: R34.2, R35.2, R46.2, U17.7 (TS)
- new net VSET: IC3.24 (VSET), R167.2
- new net VSYS: C22.2, C23.2, C25.2, D8.1 (K), IC3.19 (SYSA), IC3.6 (SYS)
Other:
- note removed: "Alternative RF Regulator B/C of 2021 Chip Shortage"
- note removed: "GPS Power"
- note removed: "L1_PROG monitors charge current using: Ichrg=988*Vprog/Rprog 3.01K = 400mA max charge current"
- note removed: "LOW = enabled Opposite polarity than other RF reg.."
- note removed: "MPPT on by default"
- note removed: "MPPT=75% Voc R11=787K, R12=121K To disable MPTT: R11=10k; R12=DNI"
- note removed: "Populating R9=107K,R10=464K sets turn-on voltage to 12V (solar input). Use this to tune efficiency"
- note removed: "Radio VDD Select"
- note removed: "VSOLAR 9V to 40V"
- note removed: "Vfloat=8.4V (2S Li-ion)"
- moved on the sheet: C32, C43, C6, Q2A, Q2B, Q3A, Q3B, R110, R15, R26, R29, R30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
