File: PyCubed/Power1.kicad_sch (KiCad schematic)
At the start: 38 parts, among them IC1 MAX1771ESA+, J3 1985807, Q1 IRLML2803, Q10 IRLML2803, Q14 MBT2222ADW1T1, Q22 NDS8434, Q23 MBT2222ADW1T1, Q24 SQS141ELNW-T1_GE3, Q25 2SC4713KT146R, Q26 2SC4713KT146R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

Commit message: PyCubed Schematic Finalized
Other:
- note added: "Value is convenient, not necessary. 10K-80K would also work for R89"
- note removed: "Value is convenient, not necessary. 10K-80K would also work for R29"
Changed lines of the file:
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@@
     (effects (font (size 0.7874 0.7874)) (justify left bottom))
   )
-  (text "Value is convenient,\nnot necessary. \n10K-80K would\nalso work for R29"
+  (text "Value is convenient,\nnot necessary. \n10K-80K would\nalso work for R89"
     (at 137.16 46.99 0)
     (effects (font (size 0.7874 0.7874)) (justify right bottom))
-  )
-  (text "Value is convenient,\nnot necessary. \n10K-80K would\nalso work for R29"
-    (at 137.16 46.99 0)
-    (effects (font (size 0.7874 0.7874)) (justify right bottom))

Commit message: PyCubed Routing Done
Connections:
- net 3V3_EN: no longer names the net of C49.2, IC1.2 (V+), Q14.6 (C1), Q26.3 (C), R106.1, R89.2
- no-connect marks 3 -> 4
Changed lines of the file:
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@@
   )
   (no_connect (at 121.92 92.71))
+  (no_connect (at 72.39 173.99))
   (no_connect (at 121.92 90.17))
   (no_connect (at 106.68 173.99))
@@
     (effects (font (size 2.159 2.159)) (justify left bottom))
   )
-  (label "3V3_EN" (at 130.81 50.8 0) (fields_autoplaced)
-    (effects (font (size 1.27 1.27)) (justify left bottom))
-  )
-  (label "3V3_EN" (at 130.81 50.8 0) (fields_autoplaced)
-    (effects (font (size 1.27 1.27)) (justify left bottom))
-  )
   (global_label "JETSON_PWR_SENSE" (shape bidirectional) (at 54.61 165.1 180)

Commit message: Mainboard Final Design
Updated BMS
Parts:
- removed C52: 10uF, Capacitor_SMD:C_0603_1608Metric, symbol Device:C_Small
- removed Q14, Q23: MBT2222ADW1T1, Package_TO_SOT_SMD:SOT-363_SC-70-6, symbol Transistor_BJT:MBT2222ADW1T1
- removed R100: 200K, Resistor_SMD:R_0603_1608Metric, symbol Device:R_US
- removed R102, R90: 100K, Resistor_SMD:R_0603_1608Metric, symbol Device:R_US
- removed R103: 10K, Resistor_SMD:R_0603_1608Metric, symbol Device:R_US
- removed R89: 73.2K, Resistor_SMD:R_0603_1608Metric, symbol Device:R_US
- removed R91: 20K, Resistor_SMD:R_0603_1608Metric, symbol Device:R_US
- added Q1: IRLML2803, mainboard:SOT-23, symbol mainboard:IRLML2803TRPBF
- added Q22: NDS8434, mainboard:NDS8434, symbol mainboard:NDS8434
- added R21: 10K, Resistor_SMD:R_0603_1608Metric, symbol mainboard:R-US_R0603
- added R22: 4.7K, Resistor_SMD:R_0603_1608Metric, symbol mainboard:R-US_R0603
- added R23: 3.3K, Resistor_SMD:R_0603_1608Metric, symbol mainboard:R-US_R0603
Connections:
- net 3.3V: now also Q22.1 (Source), Q22.2 (Source), Q22.3 (Source), R23.1
- net GND: now also Q1.2 (S), R21.2
- net at D3.4 (K_2), Q24.1 (S_1), Q24.2 (S_2)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: now also D3.2 (K_1)
- new net: Q1.1 (G), R22.2
- new net: Q1.3 (D), Q22.4 (Gate), R23.2
- new net ENAB_GPS: R21.1, R22.1
- new net GPS_PWR_IN: Q22.5 (Drain), Q22.6 (Drain), Q22.7 (Drain), Q22.8 (Drain)
- no-connect marks 4 -> 3
Other:
- note added: "GPS Power"
- note removed: ""One Shot" Regulator Reset"
- note removed: "Sets EN low dwell time"
- note removed: "Value is convenient, not necessary. 10K-80K would also work for R89"
- moved on the sheet: J3, Q1, Q22, R21, R22, R23
