File: PyCubed/RF_and_GPS.kicad_sch (KiCad schematic)
At the start: 17 parts, among them IC2 PCF8523T_1,118, J11 73412-0114, J12 73412-0114, J7 73412-0114, U10 XTB-40, U12 XTB-40, U13 EP2W+, U14 S1216V8, U20 RFM9xBreakout, U23 RFM98PW

Commit message: PyCubed Schematic Finalized
Parts:
- added C55, C56: 10nF, Capacitor_SMD:C_0603_1608Metric, symbol Device:C
- added C59: CPH3225A, CPH3225A, symbol SamacSys_Parts:CPH3225A
- added C?: 1uF, Capacitor_SMD:C_0603_1608Metric, symbol mainboard:C_Small
- added D4, D6: MBR0540T1G, SOD3716X135N, symbol SamacSys_Parts:MBR0540T1G
- added JP1, JP2, JP3, JP4, JP5, JP7: SolderJumper_2_Open, Jumper:SolderJumper-2_P1.3mm_Open_Pad1.0x1.5mm, symbol Jumper:SolderJumper_2_Open
- added Q17, Q29: BSS138DWQ-7, mainboard:BSS138DWQ-7, symbol mainboard:BSS138DWQ-7
- added Q28, Q30: MBT2222ADW1T1, Package_TO_SOT_SMD:SOT-363_SC-70-6, symbol Transistor_BJT:MBT2222ADW1T1
- added R119, R124: 200K, Resistor_SMD:R_0603_1608Metric, symbol Device:R_US
- added R120, R48: 100K, Resistor_SMD:R_0603_1608Metric, symbol Device:R_US
- added R121, R60: 680, Resistor_SMD:R_0603_1608Metric, symbol Device:R_US
- added R122, R123, R77, R78: 10K, Resistor_SMD:R_0603_1608Metric, symbol Device:R_US
- added R136, R137: ERA-8VEB1500V, ERA8KEB1004V, symbol SamacSys_Parts:ERA-8VEB1500V
Connections:
- net 3.3V: now also D4.2 (A), D6.2 (A), R120.1, R122.1, R123.1, R48.1, R77.1, R78.1
- net GND: now also C55.2, C56.2, C59.2 (-), C?.1, Q17.1 (S2), Q17.4 (S1), Q29.1 (S2), Q29.4 (S1)
- net GPS_PWR_IN: no longer U14.22 (V_BCKP)
- net RX: now also JP3.1 (A); no longer U14.20 (TXD)
- net TX: now also JP4.1 (A); no longer U14.21 (RXD)
- net VCELL: now also JP7.1 (A)
- net at U14.18 (SDA/NC): now also JP1.2 (B)
- net at U14.19 (SCL/NC): now also JP2.2 (B)
- new net: JP3.2 (B), U14.20 (TXD)
- new net: JP4.2 (B), U14.21 (RXD)
- new net: JP5.2 (B), R137.2, U14.22 (V_BCKP)
- new net: C55.1, Q17.5 (G1), R119.2
- new net: D4.1 (K), R136.1
- new net: JP7.2 (B), R136.2
- new net: Q29.6 (D1), Q30.5 (B2), R121.2, R122.2
- new net: Q28.2 (B1), R60.1
- new net: Q17.6 (D1), Q28.5 (B2), R60.2, R77.2
- new net: C56.1, Q29.5 (G1), R124.2
- new net: C59.1 (+), C?.2, JP5.1 (A)
- new net: Q30.2 (B1), R121.1
- new net: Q29.2 (G2), Q29.3 (D2), R120.2
- new net: D6.1 (K), R137.1
- new net: Q17.2 (G2), Q17.3 (D2), R48.2
- new net SCL: Q28.1 (E1), Q28.3 (C2)
- new net SCL_GPS: JP2.1 (A), Q28.4 (E2), Q28.6 (C1), R119.1, R78.2
- new net SDA: Q30.1 (E1), Q30.3 (C2)
- new net SDA_GPS: JP1.1 (A), Q30.4 (E2), Q30.6 (C1), R123.2, R124.1
- no-connect marks 42 -> 40
Other:
- note added: "I2C Bus Protection - GPS"
- moved on the sheet: C53, C?, J11, R24, U14

Commit message: PyCubed Routing Done
Parts:
- removed R54, R56: 0, Resistor_SMD:R_0805_2012Metric, symbol Device:R_US
- removed U10, U12: XTB-40, mainboard:XTB40_payload, symbol mainboard:XTB-40_payload
Connections:
- no-connect marks 40 -> 22
Other:
- note removed: "Modular Payloads"
- note removed: "PAYLOAD 1"
- note removed: "PAYLOAD 2"
- moved on the sheet: C55, C56, Q17A, Q17B, Q28A, Q28B, Q29A, Q29B, Q30A, Q30B, R119, R120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

Commit message: Mainboard Final Design
Updated BMS
Parts:
- removed U20: RFM9xBreakout, RF_Module:HOPERF_RFM9XW_SMD, symbol mainboard:RFM9xBreakout
- added C17, C18: 10uF, Capacitor_SMD:C_0603_1608Metric, symbol Device:C_Small
- added C55, C56: 10nF, Capacitor_SMD:C_0603_1608Metric, symbol Device:C
- added C65: 10uF, Capacitor_SMD:C_0603_1608Metric, symbol mainboard:10UF-0603-6.3V-20%
- added C?: 1uF, Capacitor_SMD:C_0603_1608Metric, symbol mainboard:C_Small
- added JP10: SolderJumper_2_Open, Jumper:SolderJumper-2_P1.3mm_Open_Pad1.0x1.5mm, symbol Jumper:SolderJumper_2_Open
- added Q17, Q29: BSS138DWQ-7, mainboard:BSS138DWQ-7, symbol mainboard:BSS138DWQ-7
- added Q28, Q30: MBT2222ADW1T1, Package_TO_SOT_SMD:SOT-363_SC-70-6, symbol Transistor_BJT:MBT2222ADW1T1
- added R117 (x2), R118 (x2): 0, Resistor_SMD:R_0603_1608Metric, symbol Device:R_US
- added R119, R124: 200K, Resistor_SMD:R_0603_1608Metric, symbol Device:R_US
- added R120, R48: 100K, Resistor_SMD:R_0603_1608Metric, symbol Device:R_US
- added R121, R60: 680, Resistor_SMD:R_0603_1608Metric, symbol Device:R_US
- added R122, R123, R77, R78: 10K, Resistor_SMD:R_0603_1608Metric, symbol Device:R_US
- added R15: 1K, Resistor_SMD:R_0603_1608Metric, symbol Device:R_US
- added Y2: 32.768kHz/7pF, Crystal:Crystal_SMD_MicroCrystal_CC7V-T1A-2Pin_3.2x1.5mm, symbol Device:Crystal_Small
- U14: DNI DNI -> (none)
Connections:
- net 3.3V: now also C17.2, JP10.1 (A), R120.1, R122.1, R123.1, R15.2, R48.1, R77.1, R78.1; no longer IC2.8 (VDD), U23.9 (3.3V)
- net GND: now also C17.1, C18.1, C55.2, C56.2, C65.2, C?.1, Q17.1 (S2), Q17.4 (S1), Q29.1 (S2), Q29.4 (S1)
- net SCL: now also R117.2
- net SCL_GPS: now also R117.1
- net SDA: now also R118.2
- net SDA_GPS: now also R118.1
- net at IC2.1 (OSCI): now also Y2.1
- net at IC2.2 (OSCO): now also Y2.2
- new net: Q17.2 (G2), Q17.3 (D2), R48.2
- new net: Q17.6 (D1), Q28.5 (B2), R60.2, R77.2
- new net: Q29.2 (G2), Q29.3 (D2), R120.2
- new net: C56.1, Q29.5 (G1), R124.2
- new net: C55.1, Q17.5 (G1), R119.2
- new net: C18.2, IC2.8 (VDD), R15.1
- new net: Q29.6 (D1), Q30.5 (B2), R121.2, R122.2
- new net: Q30.2 (B1), R121.1
- new net: Q28.2 (B1), R60.1
- new net P9: C65.1, C?.2, JP10.2 (B), U23.9 (3.3V)
- new net SCL2: Q28.1 (E1), Q28.3 (C2), R117.2
- new net SCL2_JETSON: Q28.4 (E2), Q28.6 (C1), R117.1, R119.1, R78.2
- new net SDA2: Q30.1 (E1), Q30.3 (C2), R118.2
- new net SDA2_JETSON: Q30.4 (E2), Q30.6 (C1), R118.1, R123.2, R124.1
- no-connect marks 22 -> 16
Other:
- moved on the sheet: C53, C55, C56, C59, C?, D4, IC2, J11, JP7, Q17A, Q17B, Q28A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
