File: Rev1/TORQUERS/Z_CAMERA_BOARD/Z_CAMERA_BOARD/Z-Axis_boards.kicad_pcb (KiCad board)
At the start: 8 copper layers, 95.9 x 90.2 mm, 34 parts, among them J1 0530470810, Q1 BSS138, Q2 BSS138, Q3 MBT2222ADW1T1, Q4 BSS138, Q5 BSS138, Q6 MBT2222ADW1T1, U1 DRV8830DGQ

Commit message: Finished Torque Coils on Camera Board 52 loops each on 2 layers
Parts:
- moved D8 77.8 mm to (247.3, 109.9)
- moved L1 77.8 mm to (238.2, 97.5)
- moved Q1 77.8 mm to (234.0, 104.2)
- moved C1 77.8 mm to (254.1, 103.3)
- moved C2 77.8 mm to (254.2, 101.6)
- moved C3 77.8 mm to (240.3, 98.1)
- moved C4 77.8 mm to (240.3, 99.9)
- moved D7 77.8 mm to (251.9, 109.9)
- moved J1 77.8 mm to (214.9, 113.1)
- moved L2 77.8 mm to (236.5, 102.8)
- moved Q2 77.8 mm to (221.3, 103.6)
- moved Q3 77.8 mm to (236.7, 96.9)
- moved Q4 77.8 mm to (226.0, 103.7)
- moved Q5 77.8 mm to (244.9, 105.1)
- moved Q6 77.8 mm to (223.7, 97.2)
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Routing:
- net /coils: track 92567.8 -> 124119.8 mm, vias 7 -> 8
