File: Rev1/USB_HUB/hub_1.kicad_sch (KiCad schematic)
At the start: 22 parts, among them IC3 USB2513B_M2, J2 826629-4, J3 826629-9, Y3 24MHZ

Commit message: USB HUB Finalized
Connections:
- net XTAL1: no longer C19.2, IC3.32 (XTALOUT), R7.1, Y3.3 (X2)
- net 1+: now reaches IC3.31 (USBDP_UP), R10.2
- net 1-: now reaches IC3.30 (USBDM_UP), R9.2
- net D_N_1 renamed D_1_N
- net D_P_1 renamed D_1_P
- new net XTAL2: C19.2, IC3.32 (XTALOUT), R7.1, Y3.3 (X2)
Changed lines of the file:
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@@
     (company "CMU")
   )
+  (junction (at 168.91 123.19) (diameter 0) (color 0 0 0 0)
+  )
+  (junction (at 158.75 50.8) (diameter 0) (color 0 0 0 0)
+  )
+  (junction (at 171.45 83.82) (diameter 0) (color 0 0 0 0)
+  )
   (junction (at 153.67 92.71) (diameter 0) (color 0 0 0 0)
   )
-  (junction (at 158.75 50.8) (diameter 0) (color 0 0 0 0)
-  )
   (junction (at 133.35 52.07) (diameter 0) (color 0 0 0 0)
   )
-  (junction (at 168.91 116.84) (diameter 0) (color 0 0 0 0)
-  )
   (junction (at 140.97 52.07) (diameter 0) (color 0 0 0 0)
   )
-  (junction (at 171.45 97.79) (diameter 0) (color 0 0 0 0)
-  )
-  (junction (at 176.53 116.84) (diameter 0) (color 0 0 0 0)
+  (junction (at 176.53 123.19) (diameter 0) (color 0 0 0 0)
   )
   (no_connect (at 105.41 123.19))
@@
     (stroke (width 0.1524) (type solid))
   )
-  (wire (pts (xy 176.53 116.84) (xy 168.91 116.84))
+  (wire (pts (xy 176.53 123.19) (xy 168.91 123.19))
+    (stroke (width 0) (type default))
+  )
+  (wire (pts (xy 176.53 106.68) (xy 176.53 123.19))
     (stroke (width 0) (type default))
   )
@@
     (stroke (width 0) (type default))
   )
-  (wire (pts (xy 171.45 83.82) (xy 171.45 97.79))
+  (wire (pts (xy 171.45 83.82) (xy 171.45 99.06))
     (stroke (width 0) (type default))
   )
@@
     (stroke (width 0) (type default))
   )
-  (wire (pts (xy 168.91 113.03) (xy 168.91 116.84))
-    (stroke (width 0.1524) (type solid))
-  )
   (wire (pts (xy 92.71 39.37) (xy 92.71 40.64))
     (stroke (width 0) (type default))
@@
     (stroke (width 0.1524) (type solid))
   )
-  (wire (pts (xy 168.91 116.84) (xy 168.91 120.65))
+  (wire (pts (xy 168.91 113.03) (xy 168.91 121.92))
     (stroke (width 0.1524) (type solid))
   )
@@
     (stroke (width 0.1524) (type solid))
   )
-  (wire (pts (xy 187.96 97.79) (xy 171.45 97.79))
+  (wire (pts (xy 171.45 83.82) (xy 189.23 83.82))
     (stroke (width 0) (type default))
   )
@@
     (stroke (width 0.1524) (type solid))
   )
+  (wire (pts (xy 168.91 123.19) (xy 168.91 125.73))
+    (stroke (width 0) (type default))
+  )
   (wire (pts (xy 77.47 58.42) (xy 77.47 62.23))
     (stroke (width 0) (type default))
@@
     (stroke (width 0.1524) (type solid))
   )
+  (wire (pts (xy 153.67 120.65) (xy 153.67 125.73))
+    (stroke (width 0) (type default))
+  )
   (wire (pts (xy 105.41 115.57) (xy 107.95 115.57))
     (stroke (width 0.1524) (type solid))
@@
     (stroke (width 0.1524) (type solid))
   )
-  (wire (pts (xy 176.53 106.68) (xy 176.53 116.84))
-    (stroke (width 0) (type default))
-  )
   (wire (pts (xy 92.71 58.42) (xy 77.47 58.42))
     (stroke (width 0) (type default))
   )
+  (wire (pts (xy 153.67 92.71) (xy 176.53 92.71))
+    (stroke (width 0) (type default))
+  )
   (wire (pts (xy 231.14 46.99) (xy 231.14 41.91))
     (stroke (width 0.1524) (type solid))
@@
     (stroke (width 0.1524) (type solid))
   )
-  (wire (pts (xy 153.67 92.71) (xy 176.53 92.71))
-    (stroke (width 0.1524) (type solid))
+  (wire (pts (xy 218.44 101.6) (xy 218.44 99.06))
+    (stroke (width 0.1524) (type solid))
+  )
+  (wire (pts (xy 105.41 128.27) (xy 107.95 128.27))
+    (stroke (width 0.1524) (type solid))
+  )
+  (wire (pts (xy 67.31 156.21) (xy 67.31 158.75))
+    (stroke (width 0.1524) (type solid))
+  )
+  (wire (pts (xy 168.91 123.19) (xy 168.91 121.92))
+    (stroke (width 0) (type default))
+  )
+  (wire (pts (xy 69.85 156.21) (xy 69.85 167.64))
+    (stroke (width 0.1524) (type solid))
+  )
+  (wire (pts (xy 168.91 99.06) (xy 171.45 99.06))
+    (stroke (width 0) (type default))
+  )
+  (wire (pts (xy 62.23 166.37) (xy 62.23 156.21))
+    (stroke (width 0) (type default))
+  )
+  (wire (pts (xy 74.93 55.88) (xy 74.93 62.23))
+    (stroke (width 0) (type default))
+  )
+  (wire (pts (xy 73.66 46.99) (xy 67.31 46.99))
+    (stroke (width 0) (type default))
+  )
+  (wire (pts (xy 105.41 107.95) (xy 113.03 107.95))
+    (stroke (width 0.1524) (type solid))
+  )
+  (wire (pts (xy 218.44 119.38) (xy 218.44 121.92))
+    (stroke (width 0.1524) (type solid))
+  )
+  (wire (pts (xy 105.41 110.49) (xy 107.95 110.49))
+    (stroke (width 0.1524) (type solid))
+  )
+  (wire (pts (xy 179.07 123.19) (xy 189.23 123.19))
+    (stroke (width 0) (type default))
   )
   (wire (pts (xy 153.67 92.71) (xy 153.67 100.33))
-    (stroke (width 0.1524) (type solid))
-  )
-  (wire (pts (xy 218.44 101.6) (xy 218.44 99.06))
-    (stroke (width 0.1524) (type solid))
-  )
-  (wire (pts (xy 105.41 128.27) (xy 107.95 128.27))
-    (stroke (width 0.1524) (type solid))
-  )
-  (wire (pts (xy 67.31 156.21) (xy 67.31 158.75))
-    (stroke (width 0.1524) (type solid))
-  )
-  (wire (pts (xy 69.85 156.21) (xy 69.85 167.64))
-    (stroke (width 0.1524) (type solid))
-  )
-  (wire (pts (xy 168.91 97.79) (xy 171.45 97.79))
-    (stroke (width 0) (type default))
-  )
-  (wire (pts (xy 62.23 166.37) (xy 62.23 156.21))
-    (stroke (width 0) (type default))
-  )
-  (wire (pts (xy 74.93 55.88) (xy 74.93 62.23))
-    (stroke (width 0) (type default))
-  )
-  (wire (pts (xy 73.66 46.99) (xy 67.31 46.99))
-    (stroke (width 0) (type default))
-  )
-  (wire (pts (xy 105.41 107.95) (xy 113.03 107.95))
-    (stroke (width 0.1524) (type solid))
-  )
-  (wire (pts (xy 176.53 116.84) (xy 176.53 123.19))
-    (stroke (width 0) (type default))
-  )
-  (wire (pts (xy 218.44 119.38) (xy 218.44 121.92))
-    (stroke (width 0.1524) (type solid))
-  )
-  (wire (pts (xy 105.41 110.49) (xy 107.95 110.49))
-    (stroke (width 0.1524) (type solid))
-  )
-  (wire (pts (xy 179.07 123.19) (xy 187.96 123.19))
     (stroke (width 0) (type default))
   )
@@
     (stroke (width 0.1524) (type solid))
   )
-  (wire (pts (xy 168.91 97.79) (xy 168.91 100.33))
-    (stroke (width 0) (type default))
-  )
-  (wire (pts (xy 187.96 123.19) (xy 187.96 97.79))
+  (wire (pts (xy 168.91 99.06) (xy 168.91 100.33))
+    (stroke (width 0) (type default))
+  )
+  (wire (pts (xy 189.23 123.19) (xy 189.23 83.82))
     (stroke (width 0) (type default))
   )
@@
     (effects (font (size 0.889 0.889)) (justify left bottom))
   )
-  (label "XTAL2" (at 171.45 92.71 0) (fields_autoplaced)
+  (label "1-" (at 82.55 58.42 0) (fields_autoplaced)
+    (effects (font (size 1.27 1.27)) (justify left bottom))
+  )
+  (label "XTAL2" (at 158.75 92.71 0) (fields_autoplaced)
     (effects (font (size 1.27 1.27)) (justify left bottom))
   )
@@
   (label "SCL/CFG0" (at 236.22 49.53 180) (fields_autoplaced)
     (effects (font (size 0.889 0.889)) (justify right bottom))
+  )
+  (label "1+" (at 76.2 55.88 0) (fields_autoplaced)
+    (effects (font (size 1.27 1.27)) (justify left bottom))
   )
   (label "SCL/CFG0" (at 107.95 115.57 0) (fields_autoplaced)
@@
     )
   )
-  (global_label "D_P_1" (shape bidirectional) (at 82.55 34.29 90) (fields_autoplaced)
+  (global_label "D_1_P" (shape bidirectional) (at 82.55 34.29 90) (fields_autoplaced)
     (effects (font (size 1.27 1.27)) (justify left))
     (property "Intersheetrefs" "${INTERSHEET_REFS}" (at 82.55 25.3218 90)
@@
     )
   )
-  (global_label "D_N_1" (shape bidirectional) (at 92.71 39.37 90) (fields_autoplaced)
+  (global_label "D_1_N" (shape bidirectional) (at 92.71 39.37 90) (fields_autoplaced)
     (effects (font (size 1.27 1.27)) (justify left))
     (property "Intersheetrefs" "${INTERSHEET_REFS}" (at 92.71 30.3413 90)
@@
     )
   )
-  (symbol (lib_id "Qwiic-USB_Hub-eagle-import:GND") (at 153.67 123.19 0) (unit 1)
-    (in_bom yes) (on_board yes) (dnp no)
-    (property "Reference" "#GND014" (at 153.67 123.19 0)
-      (effects (font (size 1.27 1.27)) hide)
-    )
-    (property "Value" "GND" (at 153.67 123.444 0)
+  (symbol (lib_id "Qwiic-USB_Hub-eagle-import:GND") (at 153.67 128.27 0) (unit 1)
+    (in_bom yes) (on_board yes) (dnp no)
+    (property "Reference" "#GND014" (at 153.67 128.27 0)
+      (effects (font (size 1.27 1.27)) hide)
+    )
+    (property "Value" "GND" (at 153.67 128.524 0)
       (effects (font (size 1.778 1.5113)) (justify top))
     )
-    (property "Footprint" "" (at 153.67 123.19 0)
-      (effects (font (size 1.27 1.27)) hide)
-    )
-    (property "Datasheet" "" (at 153.67 123.19 0)
+    (property "Footprint" "" (at 153.67 128.27 0)
+      (effects (font (size 1.27 1.27)) hide)
+    )
+    (property "Datasheet" "" (at 153.67 128.27 0)
       (effects (font (size 1.27 1.27)) hide)
     )
@@
     )
   )
-  (symbol (lib_id "Qwiic-USB_Hub-eagle-import:GND") (at 168.91 123.19 0) (unit 1)
-    (in_bom yes) (on_board yes) (dnp no)
-    (property "Reference" "#GND016" (at 168.91 123.19 0)
-      (effects (font (size 1.27 1.27)) hide)
-    )
-    (property "Value" "GND" (at 168.91 123.444 0)
+  (symbol (lib_id "Qwiic-USB_Hub-eagle-import:GND") (at 168.91 128.27 0) (unit 1)
+    (in_bom yes) (on_board yes) (dnp no)
+    (property "Reference" "#GND016" (at 168.91 128.27 0)
+      (effects (font (size 1.27 1.27)) hide)
+    )
+    (property "Value" "GND" (at 168.91 128.524 0)
       (effects (font (size 1.778 1.5113)) (justify top))
     )
-    (property "Footprint" "" (at 168.91 123.19 0)
-      (effects (font (size 1.27 1.27)) hide)
-    )
-    (property "Datasheet" "" (at 168.91 123.19 0)
-      (effects (font (size 1.27 1.27)) hide)
-    )
+    (property "Footprint" "" (at 168.91 128.27 0)
+      (effects (font (size 1.27 1.27)) hide)
+    )
+    (property "Datasheet" "" (at 168.91 128.27 0)
+      (effects (font (size 1.27 1.27)) hide)
+    )
