File: Rev1/USB_HUB/hub_2.kicad_sch (KiCad schematic)
At the start: 22 parts, among them IC4 USB2513B_M2, J1 826629-4, J5 826629-9, Y1 24MHZ

Commit message: USB HUB Finalized
Connections:
- net 2-: now reaches IC4.30 (USBDM_UP), R15.2
- net 2+: now reaches IC4.31 (USBDP_UP), R8.2
Changed lines of the file:
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@@
     (effects (font (size 0.889 0.889)) (justify right bottom))
+  )
+  (label "2+" (at 73.66 46.99 0) (fields_autoplaced)
+    (effects (font (size 1.27 1.27)) (justify left bottom))
   )
   (label "~{RESET}" (at 233.68 45.72 180) (fields_autoplaced)
@@
     (effects (font (size 0.889 0.889)) (justify right bottom))
   )
+  (label "2-" (at 78.74 49.53 0) (fields_autoplaced)
+    (effects (font (size 1.27 1.27)) (justify left bottom))
+  )
   (label "SCL/CFG0" (at 233.68 40.64 180) (fields_autoplaced)
