File: Rev1/USB_HUB/Upstream.kicad_sch (KiCad schematic)
At the start: 11 parts, among them IC1 TLV76733DGNR, IC2 TLV76733DGNR, J4 F3311A7H121014E200

Commit message: USB HUB Finalized
Connections:
- net P1+: now reaches J4.11
- net P1+: now also D3.3 (input/output_2_1); no longer D3.1 (input/output_1_1)
- net P1-: now reaches J4.10
- net P1-: now also D3.1 (input/output_1_1); no longer D3.3 (input/output_2_1)
- net P2+: now reaches D1.1 (input/output_1_1), J4.4
- net P2-: now reaches D1.3 (input/output_2_1), J4.5
- net D_N_1 renamed D_1_P
- net D_P_1 renamed D_1_N
Changed lines of the file:
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@@
     (stroke (width 0.1524) (type solid))
+  )
+  (wire (pts (xy 111.76 92.71) (xy 115.57 92.71))
+    (stroke (width 0) (type default))
   )
   (wire (pts (xy 214.63 54.61) (xy 214.63 52.07))
@@
     (stroke (width 0) (type default))
   )
+  (wire (pts (xy 115.57 87.63) (xy 115.57 74.93))
+    (stroke (width 0) (type default))
+  )
   (wire (pts (xy 151.13 62.23) (xy 151.13 64.77))
     (stroke (width 0.1524) (type solid))
@@
     (stroke (width 0.1524) (type solid))
   )
-  (wire (pts (xy 83.82 74.93) (xy 111.76 74.93))
+  (wire (pts (xy 83.82 74.93) (xy 115.57 74.93))
     (stroke (width 0) (type default))
   )
@@
     (stroke (width 0.1524) (type solid))
   )
-  (wire (pts (xy 83.82 77.47) (xy 115.57 77.47))
+  (wire (pts (xy 83.82 77.47) (xy 111.76 77.47))
     (stroke (width 0) (type default))
   )
@@
     (stroke (width 0.1524) (type solid))
   )
+  (wire (pts (xy 111.76 77.47) (xy 111.76 92.71))
+    (stroke (width 0) (type default))
+  )
   (wire (pts (xy 156.21 72.39) (xy 180.34 72.39))
     (stroke (width 0) (type default))
@@
     (stroke (width 0) (type default))
   )
-  (wire (pts (xy 115.57 77.47) (xy 115.57 87.63))
-    (stroke (width 0.1524) (type solid))
-  )
   (wire (pts (xy 220.98 120.65) (xy 220.98 118.11))
     (stroke (width 0.1524) (type solid))
@@
     (stroke (width 0) (type default))
   )
-  (wire (pts (xy 111.76 74.93) (xy 111.76 92.71))
-    (stroke (width 0.1524) (type solid))
-  )
   (wire (pts (xy 100.33 67.31) (xy 100.33 69.85))
     (stroke (width 0.1524) (type solid))
   )
   (wire (pts (xy 121.92 59.69) (xy 83.82 59.69))
-    (stroke (width 0.1524) (type solid))
-  )
-  (wire (pts (xy 111.76 92.71) (xy 115.57 92.71))
     (stroke (width 0.1524) (type solid))
   )
@@
     (effects (font (size 2.54 2.159)))
   )
-  (global_label "D_P_1" (shape bidirectional) (at 179.07 87.63 0) (fields_autoplaced)
-    (effects (font (size 1.27 1.27)) (justify left))
-    (property "Intersheetrefs" "${INTERSHEET_REFS}" (at 188.0382 87.63 0)
-      (effects (font (size 1.27 1.27)) (justify left) hide)
-    )
+  (label "P2-" (at 86.36 62.23 0) (fields_autoplaced)
+    (effects (font (size 1.27 1.27)) (justify left bottom))
+  )
+  (label "P1+" (at 97.79 77.47 0) (fields_autoplaced)
+    (effects (font (size 1.27 1.27)) (justify left bottom))
+  )
+  (label "P2+" (at 86.36 59.69 0) (fields_autoplaced)
+    (effects (font (size 1.27 1.27)) (justify left bottom))
+  )
+  (label "P1-" (at 92.71 74.93 0) (fields_autoplaced)
+    (effects (font (size 1.27 1.27)) (justify left bottom))
   )
   (global_label "5V1" (shape input) (at 184.15 90.17 0) (fields_autoplaced)
@@
     )
   )
-  (global_label "D_N_1" (shape bidirectional) (at 179.07 92.71 0) (fields_autoplaced)
-    (effects (font (size 1.27 1.27)) (justify left))
-    (property "Intersheetrefs" "${INTERSHEET_REFS}" (at 188.0987 92.71 0)
+  (global_label "D_1_N" (shape bidirectional) (at 179.07 87.63 0) (fields_autoplaced)
+    (effects (font (size 1.27 1.27)) (justify left))
+    (property "Intersheetrefs" "${INTERSHEET_REFS}" (at 188.0987 87.63 0)
       (effects (font (size 1.27 1.27)) (justify left) hide)
     )
@@
       (effects (font (size 1.27 1.27)) (justify left) hide)
     )
+  )
+  (global_label "D_1_P" (shape bidirectional) (at 179.07 92.71 0) (fields_autoplaced)
+    (effects (font (size 1.27 1.27)) (justify left))
+    (property "Intersheetrefs" "${INTERSHEET_REFS}" (at 188.0382 92.71 0)
+      (effects (font (size 1.27 1.27)) (justify left) hide)
+    )

Commit message: USB HUB Updated
Based on TA feedback
Parts:
- removed D1, D3: PRTR5V0U2F,115, PESD3V3L5UF115, symbol SamacSys_Parts:PRTR5V0U2F,115
- added U7, U8: USBLC6-2SC6, Package_TO_SOT_SMD:SOT-23-6, symbol Power_Protection:USBLC6-2SC6
Connections:
- net 5V1: now also U8.5 (VBUS)
- net 5V2: now also U7.5 (VBUS)
- net D_1_N: now also U8.6 (I/O1)
- net D_1_P: now also U8.4 (I/O2)
- net D_N_2: now also U7.4 (I/O2)
- net D_P_2: now also U7.6 (I/O1)
- net GND: now also U7.2 (GND), U8.2 (GND)
- net P1+: now also U8.3 (I/O2)
- net P1-: now also U8.1 (I/O1)
- net P2+: now also U7.1 (I/O1)
- net P2-: now also U7.3 (I/O2)
