File: Rev1/JETSON_DAUGHTER_BOARD/jetson_daughter_board/jetson_daughter_board.kicad_pcb (KiCad board)
At the start: 2 copper layers, 32.6 x 25.5 mm, 12 parts, among them J1 PYCUBED, J2 TFML-105-01-L-D-RA, J3 F3311A7H121014E200, J4 SFM-110-02-L-D-LC-K, J5 PYCUBED, J7 SFM-120-02-L-D-LC-K

Commit message: Jetson Daughter Board Updated
Added solder jumpers for i2c lines
Parts:
- removed mouse-bite-2mm-slot (x3): VAL**, Panelization:mouse-bite-2mm-slot
- added JP4: SolderJumper_2_Open, Jumper:SolderJumper-2_P1.3mm_Open_Pad1.0x1.5mm, F.Cu at (154.0, 75.0)
- added JP5: SolderJumper_2_Open, Jumper:SolderJumper-2_P1.3mm_Open_Pad1.0x1.5mm, F.Cu at (156.3, 65.1)
Connections:
- net GND2 renamed /GND2
- J7 pad 33: SCL2_JETSON_1 -> Net-(JP4-B)
- J7 pad 34: SDA2_JETSON_1 -> Net-(JP5-A)
Routing:
- net Net-(JP4-B): track 0.00 -> 5.59 mm
- net Net-(JP5-A): track 0.00 -> 3.57 mm
- net SDA2_JETSON_1: track 9.39 -> 6.71 mm
