File: Rev1/Z_PANELS/Z_PLUS/Z_PLUS_REV1/SUN_SENSOR.kicad_sch (KiCad schematic)
At the start: 34 parts, among them IC1 LTC4316IDD#PBF, Q1 BSS138, Q2 BSS138, Q4 BSS138, Q5 BSS138, U1 OPT4001DTST

Commit message: Z PLUS Updated
Parts:
- added TP1 (x2): TestPoint, TestPoint:TestPoint_Loop_D1.80mm_Drill1.0mm_Beaded, symbol Connector:TestPoint
Connections:
- net SCL_4001: now also TP1.1
- net SDA_4001: now also TP1.1
Changed lines of the file:
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@@
-    (stroke (width 0) (type default))
-  )
-  (wire (pts (xy 52.578 81.534) (xy 58.166 81.534))
     (stroke (width 0) (type default))
   )
@@
     (stroke (width 0) (type default))
   )
-  (wire (pts (xy 48.006 82.804) (xy 46.482 82.804))
+  (wire (pts (xy 48.006 82.296) (xy 46.736 82.296))
     (stroke (width 0) (type default))
   )
@@
     (stroke (width 0) (type default))
   )
-  (wire (pts (xy 48.006 82.042) (xy 48.006 82.804))
+  (wire (pts (xy 48.006 82.296) (xy 48.006 82.042))
     (stroke (width 0) (type default))
   )
@@
     (effects (font (size 1.27 1.27)) (justify left bottom))
   )
-  (label "+3.3v" (at 53.848 81.534 0) (fields_autoplaced)
+  (label "+3.3v" (at 58.166 81.534 0) (fields_autoplaced)
     (effects (font (size 1.27 1.27)) (justify left bottom))
   )
@@
     )
   )
-  (global_label "SDA_4001" (shape input) (at 46.482 82.804 180) (fields_autoplaced)
+  (global_label "SDA_4001" (shape input) (at 46.736 82.296 180) (fields_autoplaced)
     (effects (font (size 1.27 1.27)) (justify right))
-    (property "Intersheetrefs" "${INTERSHEET_REFS}" (at 34.1231 82.804 0)
+    (property "Intersheetrefs" "${INTERSHEET_REFS}" (at 34.3771 82.296 0)
       (effects (font (size 1.27 1.27)) (justify right) hide)
     )
@@
     )
   )
+  (symbol (lib_id "Connector:TestPoint") (at 45.974 69.342 0) (unit 1)
+    (in_bom yes) (on_board yes) (dnp no) (fields_autoplaced)
+    (property "Reference" "TP1" (at 48.26 64.77 0)
+      (effects (font (size 1.27 1.27)) (justify left))
+    )
+    (property "Value" "TestPoint" (at 48.26 67.31 0)
+      (effects (font (size 1.27 1.27)) (justify left))
+    )
+    (property "Footprint" "TestPoint:TestPoint_Loop_D1.80mm_Drill1.0mm_Beaded" (at 51.054 69.342 0)
+      (effects (font (size 1.27 1.27)) hide)
+    )
+    (property "Datasheet" "~" (at 51.054 69.342 0)
+      (effects (font (size 1.27 1.27)) hide)
+    )
+    (pin "1")
+    (instances
+      (project "Z_PLUS_REV1"
+        (path "/39cf28b0-d395-4333-bc0e-a98538893595/b8717c54-ec37-498b-9d48-acf0e788946a"
+          (reference "TP1") (unit 1)
+        )
+        (path "/39cf28b0-d395-4333-bc0e-a98538893595/02f51ab8-9bf5-460b-98ef-c53969a9f1c8"
+          (reference "TP3") (unit 1)
+        )
+      )
+    )
+  )
   (symbol (lib_id "power:+3.3V") (at 62.992 125.222 0) (mirror y) (unit 1)
     (in_bom yes) (on_board yes) (dnp no)
@@
     )
   )
-  (symbol (lib_id "power:+3.3V") (at 52.578 81.534 0) (mirror y) (unit 1)
-    (in_bom yes) (on_board yes) (dnp no)
-    (property "Reference" "#PWR?" (at 52.578 85.344 0)
-      (effects (font (size 1.27 1.27)) hide)
-    )
-    (property "Value" "+3.3V" (at 51.308 80.264 0)
-      (effects (font (size 1.27 1.27)) (justify left))
-    )
-    (property "Footprint" "" (at 52.578 81.534 0)
-      (effects (font (size 1.27 1.27)) hide)
-    )
-    (property "Datasheet" "" (at 52.578 81.534 0)
+  (symbol (lib_id "power:+3.3V") (at 58.166 81.534 0) (mirror y) (unit 1)
+    (in_bom yes) (on_board yes) (dnp no)
+    (property "Reference" "#PWR?" (at 58.166 85.344 0)
+      (effects (font (size 1.27 1.27)) hide)
+    )
+    (property "Value" "+3.3V" (at 56.896 80.264 0)
+      (effects (font (size 1.27 1.27)) (justify left))
+    )
+    (property "Footprint" "" (at 58.166 81.534 0)
+      (effects (font (size 1.27 1.27)) hide)
+    )
+    (property "Datasheet" "" (at 58.166 81.534 0)
       (effects (font (size 1.27 1.27)) hide)
     )
@@
         )
       )
+    )
+  )
+  (symbol (lib_id "Connector:TestPoint") (at 46.736 82.296 180) (unit 1)
+    (in_bom yes) (on_board yes) (dnp no)
+    (property "Reference" "TP1" (at 48.514 84.328 0)
+      (effects (font (size 1.27 1.27)) (justify right))
+    )
+    (property "Value" "TestPoint" (at 42.418 87.376 0)
+      (effects (font (size 1.27 1.27)) (justify right))
+    )
+    (property "Footprint" "TestPoint:TestPoint_Loop_D1.80mm_Drill1.0mm_Beaded" (at 41.656 82.296 0)
+      (effects (font (size 1.27 1.27)) hide)
+    )
+    (property "Datasheet" "~" (at 41.656 82.296 0)
+      (effects (font (size 1.27 1.27)) hide)
+    )
+    (pin "1")
+    (instances
+      (project "Z_PLUS_REV1"
+        (path "/39cf28b0-d395-4333-bc0e-a98538893595/b8717c54-ec37-498b-9d48-acf0e788946a"
+          (reference "TP1") (unit 1)
+        )
+        (path "/39cf28b0-d395-4333-bc0e-a98538893595/02f51ab8-9bf5-460b-98ef-c53969a9f1c8"
+          (reference "TP4") (unit 1)
+        )
+      )
