File: Rev1/Z_Torque_coils/Z_TORQUE_REV1/Z_TORQUE_REV1.kicad_sch (KiCad schematic)
At the start: 42 parts, among them IC1 MPM3610AGQV-Z, J1 F3311A7H121014E200, Q1 BSS138, Q2 BSS138, Q4 BSS138, Q5 BSS138, U1 DRV8830DGQ

Commit message: incremental update
Parts:
- added J2: F3311A7H121014E200, F3311A7H121014E200, symbol F3311A7H121008E200:F3311A7H121014E200
- renumbered JP4 to JP1, JP3 to JP2, JP1 to JP3, JP2 to JP4
Connections:
- net +3.3V: now also J2.10, J2.5
- net GND: now also J2.11, J2.4, J2.MP1, J2.MP2
- net SCL1_b4iso: now also J2.6, J2.9
- net SDA1_b4iso: now also J2.7, J2.8
- net VBATT: now also J1.12, J1.13, J1.2, J1.3, J2.12, J2.13, J2.2, J2.3
- net VSOLAR: now reaches J1.1
- net VSOLAR: now also J1.14, J2.1, J2.14
- no-connect marks 10 -> 4
Other:
- note added: "Stepping down voltage to 5V"
- note added: "Torque Coil driver buck"
- note removed: "Torque Coil driver boost"
- note removed: "check voltage paths put pins for vbatt"
- moved on the sheet: C1, R1, R?

Commit message: final signoff by nischal
Parts:
- C? (x2): footprint Capacitor_SMD:C_0603_1608Metric -> Capacitor_SMD:C_0201_0603Metric
- R?: footprint Resistor_SMD:R_0603_1608Metric -> Resistor_SMD:R_0805_2012Metric
Other:
- moved on the sheet: C?
Changed lines of the file:
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@@
     (stroke (width 0) (type default))
   )
-  (wire (pts (xy 141.732 40.132) (xy 141.732 37.846))
+  (wire (pts (xy 144.272 39.37) (xy 144.272 37.846))
     (stroke (width 0) (type default))
   )
@@
     (stroke (width 0) (type default))
   )
-  (wire (pts (xy 141.732 37.846) (xy 132.842 37.846))
+  (wire (pts (xy 144.272 37.846) (xy 132.842 37.846))
     (stroke (width 0) (type default))
   )
@@
     (stroke (width 0) (type default))
   )
+  (wire (pts (xy 141.732 48.006) (xy 141.732 53.594))
+    (stroke (width 0) (type default))
+  )
   (wire (pts (xy 205.486 59.69) (xy 205.486 76.2))
     (stroke (width 0) (type default))
@@
     (stroke (width 0) (type default))
   )
+  (wire (pts (xy 144.272 48.006) (xy 141.732 48.006))
+    (stroke (width 0) (type default))
+  )
   (wire (pts (xy 256.286 78.74) (xy 256.286 76.2))
     (stroke (width 0) (type default))
@@
     (stroke (width 0) (type default))
   )
-  (wire (pts (xy 141.732 47.752) (xy 141.732 53.594))
+  (wire (pts (xy 144.272 46.99) (xy 144.272 48.006))
     (stroke (width 0) (type default))
   )
@@
     )
   )
-  (symbol (lib_id "Device:C") (at 141.732 43.942 0) (unit 1)
+  (symbol (lib_id "Device:C") (at 144.272 43.18 0) (unit 1)
     (in_bom yes) (on_board yes) (dnp no)
-    (property "Reference" "C?" (at 145.034 41.656 0)
+    (property "Reference" "C?" (at 147.574 40.894 0)
       (effects (font (size 1.27 1.27)) (justify left))
     )
-    (property "Value" "0.1uF" (at 145.034 44.45 0)
+    (property "Value" "0.1uF" (at 147.574 43.688 0)
       (effects (font (size 1.27 1.27)) (justify left))
     )
-    (property "Footprint" "Capacitor_SMD:C_0805_2012Metric" (at 142.6972 47.752 0)
+    (property "Footprint" "Capacitor_SMD:C_0805_2012Metric" (at 145.2372 46.99 0)
       (effects (font (size 1.27 1.27)) hide)
     )
-    (property "Datasheet" "~" (at 141.732 43.942 0)
+    (property "Datasheet" "~" (at 144.272 43.18 0)
       (effects (font (size 1.27 1.27)) hide)
     )
@@
       (effects (font (size 1.27 1.27)) (justify right))
     )
-    (property "Footprint" "Resistor_SMD:R_0603_1608Metric" (at 75.438 134.62 90)
+    (property "Footprint" "Resistor_SMD:R_0805_2012Metric" (at 75.438 134.62 90)
       (effects (font (size 1.27 1.27)) hide)
     )
@@
       (effects (font (size 1.27 1.27)) (justify left))
     )
-    (property "Footprint" "Capacitor_SMD:C_0603_1608Metric" (at 262.3312 106.68 0)
+    (property "Footprint" "Capacitor_SMD:C_0201_0603Metric" (at 262.3312 106.68 0)
       (effects (font (size 1.27 1.27)) hide)
     )
@@
       (effects (font (size 1.27 1.27)) (justify left))
     )
-    (property "Footprint" "Capacitor_SMD:C_0603_1608Metric" (at 229.3112 106.68 0)
+    (property "Footprint" "Capacitor_SMD:C_0201_0603Metric" (at 229.3112 106.68 0)
       (effects (font (size 1.27 1.27)) hide)
     )
